Commit message: update

File: construction_model/incline_plane/urdf/incline_plane.urdf (robot description, URDF)
Before this commit: robot incline_plane, 1 links, 0 joints
Links:
- link base_link: mass 5.26740103902043 -> 39.4788577535736; geometry collision mesh filename=package://incline_plane/meshes/base_link.STL scale=5 6 8; visual mesh filename=package://incline_plane/meshes/base_link.STL scale=5 6 8
